Commit message: Fix Inertia of the model

File: omni_description/urdf/rim.xacro (robot description, xacro)
@@ -19,7 +19,7 @@
                 <origin xyz="0 0 0" rpy="0 0 0"/>
                 <mass value="${0.00835758 * scale}"/>
-                <inertia ixx="${6.63684e-07 * scale * scale}" ixy="0" ixz="0"
-                         iyy="${6.63684e-07 * scale * scale}" iyz="0"
-                         izz="${9.40333e-07 * scale * scale}"/>
+                <inertia ixx="${6.63684e-07 * scale * scale * scale * 6}" ixy="0" ixz="0"
+                         iyy="${6.63684e-07 * scale * scale * scale * 6}" iyz="0"
+                         izz="${9.40333e-07 * scale * scale * scale * 6}"/>
             </inertial>
         </link>

File: omni_description/urdf/roller.xacro (robot description, xacro)
@@ -19,7 +19,7 @@
                 <origin xyz="0.0 0.0 0.0" rpy="0.0 0.0 0.0"/>
                 <mass value="${0.00113845 * scale}"/>
-                <inertia ixx="${2.53776e-08 * scale * scale}" ixy="0" ixz="0"
-                         iyy="${2.53776e-08 * scale * scale}" iyz="0"
-                         izz="${1.47666e-08 * scale * scale}"/>
+                <inertia ixx="${2.53776e-08 * scale * scale * scale * 6}" ixy="0" ixz="0"
+                         iyy="${2.53776e-08 * scale * scale * scale * 6}" iyz="0"
+                         izz="${1.47666e-08 * scale * scale * scale * 6}"/>
             </inertial>
         </link>
